File: circuits/usb_pd_sink/usb_pd_sink.sch (KiCad schematic (older format))
At the start: 47 parts, among them J1 USB_C_Receptacle_USB2.0, J2 Conn_01x02_Female, J3 Conn_01x07_Male, Q1 DMP3013SFV, Q2 DMP3013SFV, SW1 SW_Coded, SW2 SW_Coded, U1 CYPD3177-24LQXQ

Commit message: [circuits/usb_pd_sink] Add some footprints
Parts:
- C1, C10, C11, C12, C13, C2, C3, C4, C5, C6, C7, C8, C9: footprint (none) -> Capacitor_SMD:C_0603_1608Metric
- J1: footprint (none) -> Connector_USB:USB_C_Receptacle_XKB_U262-16XN-4BVC11
- SW1, SW2: footprint (none) -> Button_Switch_SMD:Nidec_Copal_SH-7010B
- U1: footprint Cypress_Semiconductor-002-16934-0-C-* -> CYPD3177-24LQXQ:Cypress_Semiconductor-002-16934-0-C-IPC_C
Changed lines of the file:
@@
 F 0 "J1" H 1507 2517 50  0000 C CNN
 F 1 "USB_C_Receptacle_USB2.0" H 1507 2426 50  0000 C CNN
-F 2 "" H 1550 1650 50  0001 C CNN
+F 2 "Connector_USB:USB_C_Receptacle_XKB_U262-16XN-4BVC11" H 1550 1650 50  0001 C CNN
 F 3 "https://www.usb.org/sites/default/files/documents/usb_type-c.zip" H 1550 1650 50  0001 C CNN
 	1    1400 1650
@@
 F 0 "U1" H 5600 2915 50  0000 C CNN
 F 1 "CYPD3177-24LQXQ" H 5600 2824 50  0000 C CNN
-F 2 "Cypress_Semiconductor-002-16934-0-C-*" H 4550 3050 50  0001 L CNN
+F 2 "CYPD3177-24LQXQ:Cypress_Semiconductor-002-16934-0-C-IPC_C" H 4550 3050 50  0001 L CNN
 F 3 "https://www.cypress.com/file/460416/download" H 4550 3150 50  0001 L CNN
 F 4 "+105°C" H 4550 3250 50  0001 L CNN "ambient temperature range high"
@@
 F 0 "SW1" H 2032 6825 50  0000 C CNN
 F 1 "SW_Coded" H 2032 6734 50  0000 C CNN
-F 2 "" H 1875 6375 50  0001 C CNN
+F 2 "Button_Switch_SMD:Nidec_Copal_SH-7010B" H 1875 6375 50  0001 C CNN
 F 3 "~" H 1875 6375 50  0001 C CNN
 	1    1900 6350
@@
 F 0 "SW2" H 6920 6325 50  0000 R CNN
 F 1 "SW_Coded" H 6920 6234 50  0000 R CNN
-F 2 "" H 7175 6275 50  0001 C CNN
+F 2 "Button_Switch_SMD:Nidec_Copal_SH-7010B" H 7175 6275 50  0001 C CNN
 F 3 "~" H 7175 6275 50  0001 C CNN
 	1    7200 6250
@@
 F 0 "C4" H 2950 1400 50  0000 L CNN
 F 1 "3.3u" H 3050 1200 50  0000 L CNN
-F 2 "" H 3088 1150 50  0001 C CNN
+F 2 "Capacitor_SMD:C_0603_1608Metric" H 3088 1150 50  0001 C CNN
 F 3 "~" H 3050 1300 50  0001 C CNN
 	1    3050 1300
@@
 F 0 "C1" H 2550 1400 50  0000 L CNN
 F 1 "47n" H 2500 1200 50  0000 L CNN
-F 2 "" H 2688 1150 50  0001 C CNN
+F 2 "Capacitor_SMD:C_0603_1608Metric" H 2688 1150 50  0001 C CNN
 F 3 "~" H 2650 1300 50  0001 C CNN
 	1    2650 1300
@@
 F 0 "C6" H 3615 1296 50  0000 L CNN
 F 1 "1u" H 3615 1205 50  0000 L CNN
-F 2 "" H 3538 1100 50  0001 C CNN
+F 2 "Capacitor_SMD:C_0603_1608Metric" H 3538 1100 50  0001 C CNN
 F 3 "~" H 3500 1250 50  0001 C CNN
 	1    3500 1250
@@
 F 0 "C2" H 2650 4100 50  0000 L CNN
 F 1 "390p" H 2550 3900 50  0000 L CNN
-F 2 "" H 2788 3850 50  0001 C CNN
+F 2 "Capacitor_SMD:C_0603_1608Metric" H 2788 3850 50  0001 C CNN
 F 3 "~" H 2750 4000 50  0001 C CNN
 	1    2750 4000
@@
 F 0 "C5" H 3000 4100 50  0000 L CNN
 F 1 "390p" H 3100 3900 50  0000 L CNN
-F 2 "" H 3138 3850 50  0001 C CNN
+F 2 "Capacitor_SMD:C_0603_1608Metric" H 3138 3850 50  0001 C CNN
 F 3 "~" H 3100 4000 50  0001 C CNN
 	1    3100 4000
@@
 F 0 "C7" H 3615 4046 50  0000 L CNN
 F 1 "1u" H 3615 3955 50  0000 L CNN
-F 2 "" H 3538 3850 50  0001 C CNN
+F 2 "Capacitor_SMD:C_0603_1608Metric" H 3538 3850 50  0001 C CNN
 F 3 "~" H 3500 4000 50  0001 C CNN
 	1    3500 4000
@@
 F 0 "C8" H 4900 2200 50  0000 L CNN
 F 1 "1u" H 4850 2000 50  0000 L CNN
-F 2 "" H 5038 1950 50  0001 C CNN
+F 2 "Capacitor_SMD:C_0603_1608Metric" H 5038 1950 50  0001 C CNN
 F 3 "~" H 5000 2100 50  0001 C CNN
 	1    5000 2100
@@
 F 0 "C9" H 5100 2200 50  0000 L CNN
 F 1 "0.1u" H 5100 2000 50  0000 L CNN
-F 2 "" H 5238 1950 50  0001 C CNN
+F 2 "Capacitor_SMD:C_0603_1608Metric" H 5238 1950 50  0001 C CNN
 F 3 "~" H 5200 2100 50  0001 C CNN
 	1    5200 2100
@@
 F 0 "C10" H 5400 2200 50  0000 L CNN
 F 1 "0.1u" H 5400 2000 50  0000 L CNN
-F 2 "" H 5438 1950 50  0001 C CNN
+F 2 "Capacitor_SMD:C_0603_1608Metric" H 5438 1950 50  0001 C CNN
 F 3 "~" H 5400 2100 50  0001 C CNN
 	1    5400 2100
@@
 F 0 "C11" H 5650 1350 50  0000 L CNN
 F 1 "0.1u" H 5650 1150 50  0000 L CNN
-F 2 "" H 5838 1100 50  0001 C CNN
+F 2 "Capacitor_SMD:C_0603_1608Metric" H 5838 1100 50  0001 C CNN
 F 3 "~" H 5800 1250 50  0001 C CNN
 	1    5800 1250
@@
 F 0 "C12" H 5850 1350 50  0000 L CNN
 F 1 "1u" H 5900 1150 50  0000 L CNN
-F 2 "" H 6038 1100 50  0001 C CNN
+F 2 "Capacitor_SMD:C_0603_1608Metric" H 6038 1100 50  0001 C CNN
 F 3 "~" H 6000 1250 50  0001 C CNN
 	1    6000 1250
@@
 F 0 "C13" H 6200 1350 50  0000 L CNN
 F 1 "10u" H 6200 1150 50  0000 L CNN
-F 2 "" H 6238 1100 50  0001 C CNN
+F 2 "Capacitor_SMD:C_0603_1608Metric" H 6238 1100 50  0001 C CNN
 F 3 "~" H 6200 1250 50  0001 C CNN
 	1    6200 1250
@@
 F 0 "C3" H 2750 1400 50  0000 L CNN
 F 1 "0.47u" H 2750 1200 50  0000 L CNN
-F 2 "" H 2888 1150 50  0001 C CNN
+F 2 "Capacitor_SMD:C_0603_1608Metric" H 2888 1150 50  0001 C CNN
 F 3 "~" H 2850 1300 50  0001 C CNN
 	1    2850 1300
